File: esp32-nfc-reader/esp32-nfc-reader.kicad_pcb (KiCad board)
At the start: 4 copper layers, 46 x 89.5 mm, 55 parts, among them J1 USB_C_Receptacle_USB2.0_16P, J2 Conn_01x02_Pin, J3 Conn_01x08, K1 Relay_SPDT, Q1 PMOS, Q2 Q_NMOS, SW1 RESET, SW2 BOOT, SW3 USER_INPUT, U1 ESP32-S3-WROOM-1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

Commit message: added antenna loop
Parts:
- removed AE1: Antenna, Connector_PinSocket_2.54mm:PinSocket_1x01_P2.54mm_Vertical
- added AE2: Antenna_Loop, RF_Antenna:Coilcraft_MA5532-AE_RFID, F.Cu at (131.0, 90.8)
Connections:
- net /RX renamed Net-(U3-RX)
- C8 pad 2: Net-(AE1-A) -> Net-(AE2-Pad1)
- C9 pad 1: Net-(AE1-A) -> Net-(AE2-Pad2)
Routing:
- net Net-(AE2-Pad2): track 0.00 -> 21.4 mm, vias 0 -> 2
- net Net-(AE2-Pad1): track 0.00 -> 10.8 mm
- net Net-(AE1-A): track 5.93 -> 0.00 mm
